Commit message: Change to actual dimensions

File: urdf/d2rbot.urdf.xacro (robot description, xacro)
@@ -13,7 +13,4 @@
   <material name="white">
     <color rgba="1 1 1 1"/>
-  </material>
-  <material name="paua-blue">
-    <color rgba="0.145 0.161 0.345 1"/>
   </material>
   <material name="shark-blue">
@@ -34,5 +31,6 @@
   <xacro:property name="motor_width" value="0.023" />
   <xacro:property name="motor_height" value="0.038" />
-  <xacro:property name="motor_offset" value="0.0465" />
+  <xacro:property name="motor_x_offset" value="0.0215" />
+  <xacro:property name="motor_y_offset" value="0.0465" />
   <xacro:property name="motorshaft_x_offset" value="0.0215" />
   <xacro:property name="motorshaft_y_offset" value="${motor_width/2}" />
@@ -49,4 +47,6 @@
   <xacro:property name="connector_x_offset" value="0.060" />
   <xacro:property name="connector_y_offset" value="0.040" />
+  <xacro:property name="connector_y_narrow_compensation" value="0.020" />
+  <xacro:property name="connector_y_wide_compensation" value="0.000" />
   <xacro:property name="connector_mass" value="0.001" />
   <!-- Empty first link "world" -->
@@ -99,5 +99,4 @@
           <box size="${motor_length} ${motor_width} ${motor_height}"/>
         </geometry>
-        <!--  <origin xyz="${motor_length/2} ${motor_width/2} ${motor_height/2}" rpy="0.0 0.0 0.0"/>  -->
         <origin xyz="0.0 0.0 0.0" rpy="0.0 0.0 0.0"/>
         <material name="${materialname}"/>
@@ -113,5 +112,5 @@
       <parent link="${parent}_link"/>
       <child link="${prefix}motorblock_link"/>
-      <origin xyz="0.0 ${reflect*(motor_offset - motor_width/2)} ${motor_height/2 + plate_height/2}"/>
+      <origin xyz="${-1*motor_x_offset} ${reflect*(motor_y_offset - motor_width/2)} ${motor_height/2 + plate_height/2}"/>
     </joint>
   </xacro:macro>
@@ -143,5 +142,5 @@
   <!-- Note: connectors are for visual display only. -->
   <!--       The three plates are directly joint to each other.-->
-  <xacro:macro name="connector" params="prefix materialname x_reflect y_reflect parent">
+  <xacro:macro name="connector" params="prefix materialname x_reflect y_reflect y_compensation parent">
     <link name="${prefix}_${parent}connector_link">
       <visual>
@@ -161,5 +160,5 @@
       <parent link="${parent}_link"/>
       <child link="${prefix}_${parent}connector_link"/>
-      <origin xyz="${x_reflect * connector_x_offset} ${y_reflect * connector_y_offset} ${connector_height/2}"/>
+      <origin xyz="${x_reflect * connector_x_offset} ${y_reflect * (connector_y_offset - y_compensation)} ${connector_height/2}"/>
     </joint>
   </xacro:macro>
@@ -180,18 +179,18 @@
   <xacro:wheel prefix="right" reflect="-1" materialname="dark_gray" parent="rightmotorblock" />
   <!-- Forwardleft connector bottomplate -->
-  <xacro:connector prefix="forwardleft" x_reflect="1" y_reflect="1" materialname="paua-blue" parent="bottomplate" />
+  <xacro:connector prefix="forwardleft" x_reflect="1" y_reflect="1" y_compensation="${connector_y_wide_compensation}" materialname="shark-blue" parent="bottomplate" />
   <!-- Forwardright connector bottomplate -->
-  <xacro:connector prefix="forwardright" x_reflect="1" y_reflect="-1" materialname="paua-blue" parent="bottomplate" />
+  <xacro:connector prefix="forwardright" x_reflect="1" y_reflect="-1" y_compensation="${connector_y_wide_compensation}" materialname="shark-blue" parent="bottomplate" />
   <!-- Backwardleft connector bottomplate -->
-  <xacro:connector prefix="backwardleft" x_reflect="-1" y_reflect="1" materialname="shark-blue" parent="bottomplate" />
+  <xacro:connector prefix="backwardleft" x_reflect="-1" y_reflect="1" y_compensation="${connector_y_narrow_compensation}" materialname="shark-blue" parent="bottomplate" />
   <!-- Backwardright connector bottomplate -->
-  <xacro:connector prefix="backwardright" x_reflect="-1" y_reflect="-1" materialname="shark-blue" parent="bottomplate" />
+  <xacro:connector prefix="backwardright" x_reflect="-1" y_reflect="-1" y_compensation="${connector_y_narrow_compensation}" materialname="shark-blue" parent="bottomplate" />
   <!-- Forwardleft connector niddleplate -->
-  <xacro:connector prefix="forwardleft" x_reflect="1" y_reflect="1" materialname="paua-blue" parent="middleplate" />
+  <xacro:connector prefix="forwardleft" x_reflect="1" y_reflect="1" y_compensation="${connector_y_narrow_compensation}" materialname="shark-blue" parent="middleplate" />
   <!-- Forwardright connector middleplate -->
-  <xacro:connector prefix="forwardright" x_reflect="1" y_reflect="-1" materialname="paua-blue" parent="middleplate" />
+  <xacro:connector prefix="forwardright" x_reflect="1" y_reflect="-1" y_compensation="${connector_y_narrow_compensation}" materialname="shark-blue" parent="middleplate" />
   <!-- Backwardleft connector middleplate -->
-  <xacro:connector prefix="backwardleft" x_reflect="-1" y_reflect="1" materialname="shark-blue" parent="middleplate" />
+  <xacro:connector prefix="backwardleft" x_reflect="-1" y_reflect="1" y_compensation="${connector_y_wide_compensation}" materialname="shark-blue" parent="middleplate" />
   <!-- Backwardright connector middleplate -->
-  <xacro:connector prefix="backwardright" x_reflect="-1" y_reflect="-1" materialname="shark-blue" parent="middleplate" />
+  <xacro:connector prefix="backwardright" x_reflect="-1" y_reflect="-1" y_compensation="${connector_y_wide_compensation}" materialname="shark-blue" parent="middleplate" />
 </robot>

Commit message: Use default value in macro-param of connector xacro-macro

File: urdf/d2rbot.urdf.xacro (robot description, xacro)
@@ -47,6 +47,5 @@
   <xacro:property name="connector_x_offset" value="0.060" />
   <xacro:property name="connector_y_offset" value="0.040" />
-  <xacro:property name="connector_y_narrow_compensation" value="0.020" />
-  <xacro:property name="connector_y_wide_compensation" value="0.000" />
+  <xacro:property name="connector_y_narrow_shift" value="-0.020" />
   <xacro:property name="connector_mass" value="0.001" />
   <!-- Empty first link "world" -->
@@ -142,5 +141,5 @@
   <!-- Note: connectors are for visual display only. -->
   <!--       The three plates are directly joint to each other.-->
-  <xacro:macro name="connector" params="prefix materialname x_reflect y_reflect y_compensation parent">
+  <xacro:macro name="connector" params="prefix materialname x_reflect y_reflect y_shift:=0.000 parent">
     <link name="${prefix}_${parent}connector_link">
       <visual>
@@ -160,5 +159,5 @@
       <parent link="${parent}_link"/>
       <child link="${prefix}_${parent}connector_link"/>
-      <origin xyz="${x_reflect * connector_x_offset} ${y_reflect * (connector_y_offset - y_compensation)} ${connector_height/2}"/>
+      <origin xyz="${x_reflect * connector_x_offset} ${y_reflect * (connector_y_offset + y_shift)} ${connector_height/2}"/>
     </joint>
   </xacro:macro>
@@ -179,18 +178,18 @@
   <xacro:wheel prefix="right" reflect="-1" materialname="dark_gray" parent="rightmotorblock" />
   <!-- Forwardleft connector bottomplate -->
-  <xacro:connector prefix="forwardleft" x_reflect="1" y_reflect="1" y_compensation="${connector_y_wide_compensation}" materialname="shark-blue" parent="bottomplate" />
+  <xacro:connector prefix="forwardleft" x_reflect="1" y_reflect="1" materialname="shark-blue" parent="bottomplate" />
   <!-- Forwardright connector bottomplate -->
-  <xacro:connector prefix="forwardright" x_reflect="1" y_reflect="-1" y_compensation="${connector_y_wide_compensation}" materialname="shark-blue" parent="bottomplate" />
+  <xacro:connector prefix="forwardright" x_reflect="1" y_reflect="-1" materialname="shark-blue" parent="bottomplate" />
   <!-- Backwardleft connector bottomplate -->
-  <xacro:connector prefix="backwardleft" x_reflect="-1" y_reflect="1" y_compensation="${connector_y_narrow_compensation}" materialname="shark-blue" parent="bottomplate" />
+  <xacro:connector prefix="backwardleft" x_reflect="-1" y_reflect="1" y_shift="${connector_y_narrow_shift}" materialname="shark-blue" parent="bottomplate" />
   <!-- Backwardright connector bottomplate -->
-  <xacro:connector prefix="backwardright" x_reflect="-1" y_reflect="-1" y_compensation="${connector_y_narrow_compensation}" materialname="shark-blue" parent="bottomplate" />
+  <xacro:connector prefix="backwardright" x_reflect="-1" y_reflect="-1" y_shift="${connector_y_narrow_shift}" materialname="shark-blue" parent="bottomplate" />
   <!-- Forwardleft connector niddleplate -->
-  <xacro:connector prefix="forwardleft" x_reflect="1" y_reflect="1" y_compensation="${connector_y_narrow_compensation}" materialname="shark-blue" parent="middleplate" />
+  <xacro:connector prefix="forwardleft" x_reflect="1" y_reflect="1" y_shift="${connector_y_narrow_shift}" materialname="shark-blue" parent="middleplate" />
   <!-- Forwardright connector middleplate -->
-  <xacro:connector prefix="forwardright" x_reflect="1" y_reflect="-1" y_compensation="${connector_y_narrow_compensation}" materialname="shark-blue" parent="middleplate" />
+  <xacro:connector prefix="forwardright" x_reflect="1" y_reflect="-1" y_shift="${connector_y_narrow_shift}" materialname="shark-blue" parent="middleplate" />
   <!-- Backwardleft connector middleplate -->
-  <xacro:connector prefix="backwardleft" x_reflect="-1" y_reflect="1" y_compensation="${connector_y_wide_compensation}" materialname="shark-blue" parent="middleplate" />
+  <xacro:connector prefix="backwardleft" x_reflect="-1" y_reflect="1" materialname="shark-blue" parent="middleplate" />
   <!-- Backwardright connector middleplate -->
-  <xacro:connector prefix="backwardright" x_reflect="-1" y_reflect="-1" y_compensation="${connector_y_wide_compensation}" materialname="shark-blue" parent="middleplate" />
+  <xacro:connector prefix="backwardright" x_reflect="-1" y_reflect="-1" materialname="shark-blue" parent="middleplate" />
 </robot>

Commit message: Change mass of plates , wheel , motors and connectors

File: urdf/d2rbot.urdf.xacro (robot description, xacro)
@@ -24,5 +24,6 @@
   <xacro:property name="plate_diameter" value="0.160" />
   <xacro:property name="plate_height" value="0.0025" />
-  <xacro:property name="plate_mass" value="0.392" />
+  <xacro:property name="plate_mass" value="0.394" />
+  <xacro:property name="bottomplate_mass" value="0.350" />
   <xacro:property name="distance_between_plates" value="${connector_height + plate_height}" />
   <!-- Properties of the motors -->
@@ -36,10 +37,10 @@
   <xacro:property name="motorshaft_y_offset" value="${motor_width/2}" />
   <xacro:property name="motorshaft_z_offset" value="-0.0190" />
-  <xacro:property name="motor_mass" value="0.029" />
+  <xacro:property name="motor_mass" value="0.037" />
   <!--- Properties of the wheels -->
   <xacro:property name="wheel_diameter" value="0.065" />
   <xacro:property name="wheel_width" value="0.006" />
   <xacro:property name="wheel_offset" value="0.007" />
-  <xacro:property name="wheel_mass" value="0.011" />
+  <xacro:property name="wheel_mass" value="0.012" />
   <!-- Properties of the vertical connection beams -->
   <xacro:property name="connector_height" value="0.055" />
@@ -48,5 +49,5 @@
   <xacro:property name="connector_y_offset" value="0.040" />
   <xacro:property name="connector_y_narrow_shift" value="-0.020" />
-  <xacro:property name="connector_mass" value="0.001" />
+  <xacro:property name="connector_mass" value="0.002" />
   <!-- Empty first link "world" -->
   <link name="world" />
@@ -70,5 +71,5 @@
   <xacro:include filename="$(find d2rbot_description)/urdf/default_inertial.urdf.xacro"/>
   <!-- Start plate macro -->
-  <xacro:macro name="plate" params="prefix materialname parent parentdistance">
+  <xacro:macro name="plate" params="prefix materialname mass parent parentdistance">
     <link name="${prefix}plate_link">
       <visual>
@@ -83,5 +84,5 @@
         </geometry>
       </collision>
-      <xacro:default_cylinder_inertial mass="${plate_mass}" radius="${plate_diameter/2}" height="${plate_height}" />
+      <xacro:default_cylinder_inertial mass="${mass}" radius="${plate_diameter/2}" height="${plate_height}" />
     </link>
     <joint name="${parent}_to_${prefix}plate_joint" type="fixed">
@@ -164,9 +165,9 @@
   <!-- Start of the actual robot model -->
   <!-- Bottomplate -->
-  <xacro:plate prefix="bottom" materialname="black" parent="base" parentdistance="${chassis_z_offset}"/>
+  <xacro:plate prefix="bottom" materialname="black" mass="${bottomplate_mass}" parent="base" parentdistance="${chassis_z_offset}"/>
   <!-- Middleplate -->
-  <xacro:plate prefix="middle" materialname="orange" parent="bottomplate" parentdistance="${distance_between_plates}"/>
+  <xacro:plate prefix="middle" materialname="orange" mass="${plate_mass}" parent="bottomplate" parentdistance="${distance_between_plates}"/>
   <!-- Topplate -->
-  <xacro:plate prefix="top" materialname="orange" parent="middleplate" parentdistance="${distance_between_plates}"/>
+  <xacro:plate prefix="top" materialname="orange" mass="${plate_mass}" parent="middleplate" parentdistance="${distance_between_plates}"/>
   <!-- Leftmotorblock -->
   <xacro:motorblock prefix="left" reflect="1" materialname="yellow" parent="bottomplate" />
