Commit message: Update C1 urdf.xacro: use fixed values instead of variables

File: urdf/rplidar_c1.urdf.xacro (robot description, xacro)
@@ -3,13 +3,6 @@
   <!-- TODO  check if works as an include -->
   <material name="C1_black">
-    <color rgba="0 0 0 1"/>
+    <color rgba="0 0 0 0.4"/>
   </material>
-  <!-- Properties C1 -->
-  <xacro:property name="C1_box_length" value="0.0550" />
-  <xacro:property name="C1_box_width" value="0.0550" />
-  <xacro:property name="C1_box_height" value="0.0253" />
-  <xacro:property name="C1_cylinder_diameter" value="0.0520" />
-  <xacro:property name="C1_cylinder_heigth" value="0.0182" />
-  <xacro:property name="C1_mass" value="0.096" />
   <!-- Empty first link "world" -->
   <link name="world" />
@@ -33,26 +26,35 @@
   <xacro:include filename="$(find d2rbot_description)/urdf/default_inertial.urdf.xacro"/>
   <!-- C1 lidar macro -->
-  <xacro:macro name="C1-lidar" params="prefix materialname parent">
+  <xacro:macro name="C1-lidar" params="prefix parent">
+    <!-- Properties C1       -->
+    <!-- Box                 -->
+    <!--   length   : 0,0550 -->
+    <!--   width    : 0,0550 -->
+    <!--   height   : 0,0253 -->
+    <!-- Cylinder         -->
+    <!--   diameter : 0.0520 -->
+    <!--   height   : 0,0182 -->
+    <!-- Mass : 0.096        -->
     <link name="${prefix}_link">
       <visual>
         <geometry>
-          <box size="${C1_box_length} ${C1_box_width} ${C1_box_height}"/>
+          <box size="0.0550 0.0550 0.0253"/>
         </geometry>
-        <origin xyz="0.0 0.0 ${C1_box_height/2}" rpy="0.0 0.0 0.0"/>
-        <material name="${materialname}"/>
+        <origin xyz="0.0 0.0 ${0.0253/2}" rpy="0.0 0.0 0.0"/>
+        <material name="C1_black"/>
       </visual>
       <visual>
-        <origin xyz="0 0 ${C1_box_height + (C1_cylinder_heigth/2)}" rpy="0 0 0" />
+        <origin xyz="0 0 ${0.0253 + (0.0182/2)}" rpy="0 0 0" />
         <geometry>
-          <cylinder length="${C1_cylinder_heigth}" radius="${C1_cylinder_diameter/2}"/>
+          <cylinder length="0.0182" radius="${0.0520/2}"/>
         </geometry>
-        <material name="${materialname}"/>
+        <material name="C1_black"/>
       </visual>
       <collision>
         <geometry>
-          <box size="${C1_box_length} ${C1_box_width} ${C1_box_height + C1_cylinder_heigth}"/>
+          <box size="0.0550 0.0550 ${0.0253 + 0.0182}"/>
         </geometry>
       </collision>
-      <xacro:default_box_inertial mass="${C1_mass}" />
+      <xacro:default_box_inertial mass="0.096" />
     </link>
     <joint name="${parent}_to_${prefix}_joint" type="fixed">
@@ -63,4 +65,4 @@
   </xacro:macro>
   <!-- Start of the actual C1 lidar -->
-  <xacro:C1-lidar prefix="unique" materialname="C1_black" parent="base"/>
+  <xacro:C1-lidar prefix="unique" parent="base"/>
 </robot>
